File: schema/dtz80-complete/dtz80-complete.sch (KiCad schematic (older format))
At the start: 52 parts, among them IC1 Z80SIO, IC2 Z80CTC, J1 FT_232, J1_5VtoSerial1 Conn_01x02, J2 CTC, J3 8 Bit Port, J4 PS/2 Keyboard, J5 RC2014Bus, Q1 NPN, Q2 NPN, U1 74LS32, U10 5161AS, U11 HM62256, U12 74HC245, U2 Z80CPU, U3 28C256, U4 74LS393, U5 74LS04, U6 74LS138, U7 74LS573, U8 74HC245, U9 74LS04, X1 CXO_DIP8, Y1 Crystal

Commit message: reset circuit
Parts:
- added C?: 100nF, symbol Device:C
- added C?: 10nF, symbol Device:C
- added C?: 10uF, symbol Device:CP
- added R?: 47K, symbol Device:R
- added R?: 1M, symbol Device:R
- added SW?: Reset, symbol Switch:SW_MEC_5G
- added U?: NE555P, Package_DIP:DIP-8_W7.62mm, symbol Timer:NE555P
Connections:
- net labels added: TODO_INVERT_RESET
- wire segments 388 -> 419
- no-connect marks 31 -> 30
Changed lines of the file:
@@
 	1    0    0    -1
 $EndComp
-Wire Wire Line
-	10000 2350 10000 2200
 $Comp
 L power:+5V #PWR025
@@
 Text Label 8900 5050 0    50   ~ 0
 A1
-NoConn ~ 10050 2050
 Text Label 12300 2950 0    50   ~ 0
 D0
@@
 Text Label 7200 4250 0    50   ~ 0
 VCC
+$Comp
+L Timer:NE555P U?
+U 1 1 607E50E5
+P 11750 1150
+F 0 "U?" H 11750 1731 50  0000 C CNN
+F 1 "NE555P" H 11750 1640 50  0000 C CNN
+F 2 "Package_DIP:DIP-8_W7.62mm" H 12400 750 50  0001 C CNN
+F 3 "http://www.ti.com/lit/ds/symlink/ne555.pdf" H 12600 750 50  0001 C CNN
+	1    11750 1150
+	1    0    0    -1
+$EndComp
+$Comp
+L power:+5V #PWR?
+U 1 1 607EA290
+P 11750 150
+F 0 "#PWR?" H 11750 0   50  0001 C CNN
+F 1 "+5V" H 11765 323 50  0000 C CNN
+F 2 "" H 11750 150 50  0001 C CNN
+F 3 "" H 11750 150 50  0001 C CNN
+	1    11750 150
+	1    0    0    -1
+$EndComp
+$Comp
+L power:GND #PWR?
+U 1 1 607EA9EB
+P 11750 1950
+F 0 "#PWR?" H 11750 1700 50  0001 C CNN
+F 1 "GND" H 11755 1777 50  0000 C CNN
+F 2 "" H 11750 1950 50  0001 C CNN
+F 3 "" H 11750 1950 50  0001 C CNN
+	1    11750 1950
+	1    0    0    -1
+$EndComp
+$Comp
+L Device:C C?
+U 1 1 607EB630
+P 10600 1300
+F 0 "C?" H 10715 1346 50  0000 L CNN
+F 1 "100nF" H 10715 1255 50  0000 L CNN
+F 2 "" H 10638 1150 50  0001 C CNN
+F 3 "~" H 10600 1300 50  0001 C CNN
+	1    10600 1300
+	1    0    0    -1
+$EndComp
+$Comp
+L Device:C C?
+U 1 1 607EC0A9
+P 11350 1750
+F 0 "C?" H 11465 1796 50  0000 L CNN
+F 1 "10nF" H 11465 1705 50  0000 L CNN
+F 2 "" H 11388 1600 50  0001 C CNN
+F 3 "~" H 11350 1750 50  0001 C CNN
+	1    11350 1750
+	1    0    0    -1
+$EndComp
+$Comp
+L Switch:SW_MEC_5G SW?
+U 1 1 607EDE72
+P 10300 950
+F 0 "SW?" H 10300 1235 50  0000 C CNN
+F 1 "Reset" H 10300 1144 50  0000 C CNN
+F 2 "" H 10300 1150 50  0001 C CNN
+F 3 "http://www.apem.com/int/index.php?controller=attachment&id_attachment=488" H 10300 1150 50  0001 C CNN
+	1    10300 950
+	1    0    0    -1
+$EndComp
+$Comp
+L Device:CP C?
+U 1 1 607EEEB1
+P 12550 1600
+F 0 "C?" H 12433 1554 50  0000 R CNN
+F 1 "10uF" H 12433 1645 50  0000 R CNN
+F 2 "" H 12588 1450 50  0001 C CNN
+F 3 "~" H 12550 1600 50  0001 C CNN
+	1    12550 1600
+	1    0    0    1
+$EndComp
+Wire Wire Line
+	11750 1550 11750 1950
+Wire Wire Line
+	12550 1750 12550 1950
+Wire Wire Line
+	12550 1950 11750 1950
+Connection ~ 11750 1950
+Wire Wire Line
+	12550 1450 12550 1350
+Wire Wire Line
+	12550 1350 12250 1350
+Wire Wire Line
+	12550 1350 12550 1150
+Wire Wire Line
+	12550 1150 12250 1150
+Connection ~ 12550 1350
+Wire Wire Line
+	12550 1150 12550 650
+Connection ~ 12550 1150
+$Comp
+L Device:R R?
+U 1 1 60938BA3
+P 12550 500
+F 0 "R?" H 12620 546 50  0000 L CNN
+F 1 "47K" H 12620 455 50  0000 L CNN
+F 2 "" V 12480 500 50  0001 C CNN
+F 3 "~" H 12550 500 50  0001 C CNN
+	1    12550 500
+	1    0    0    -1
+$EndComp
+Wire Wire Line
+	12550 350  12550 150
+Wire Wire Line
+	12550 150  11750 150
+Wire Wire Line
+	12250 950  12800 950
+Wire Wire Line
+	11250 950  10600 950
+Wire Wire Line
+	10100 950  10100 1650
+Wire Wire Line
+	10100 1650 10600 1650
+Wire Wire Line
+	11150 1650 11150 1950
+Wire Wire Line
+	11150 1950 11350 1950
+Wire Wire Line
+	11250 1150 11100 1150
+Wire Wire Line
+	11100 1150 11100 1600
+Wire Wire Line
+	11100 1600 11350 1600
+Wire Wire Line
+	11350 1900 11350 1950
+Connection ~ 11350 1950
+Wire Wire Line
+	11350 1950 11750 1950
+Wire Wire Line
+	11750 150  11000 150
+Wire Wire Line
+	10600 150  10600 400
+Connection ~ 11750 150
+$Comp
+L Device:R R?
+U 1 1 60A8A53F
+P 10600 550
+F 0 "R?" H 10670 596 50  0000 L CNN
+F 1 "1M" H 10670 505 50  0000 L CNN
+F 2 "" V 10530 550 50  0001 C CNN
+F 3 "~" H 10600 550 50  0001 C CNN
+	1    10600 550
+	1    0    0    -1
+$EndComp
+Wire Wire Line
+	10600 700  10600 950
+Connection ~ 10600 950
+Wire Wire Line
+	10600 950  10500 950
+Wire Wire Line
+	10600 950  10600 1150
+Wire Wire Line
+	10600 1450 10600 1650
+Connection ~ 10600 1650
+Wire Wire Line
+	10600 1650 11150 1650
+Wire Wire Line
+	11250 1350 11000 1350
+Wire Wire Line
+	11000 1350 11000 150
+Connection ~ 11000 150
+Wire Wire Line
+	11000 150  10600 150
+Wire Wire Line
+	10000 2200 10000 2350
+Text Label 12700 950  0    50   ~ 0
+TODO_INVERT_RESET
 $EndSCHEMATC

Commit message: schema, datasheets etc
Parts:
- removed J4: PS/2 Keyboard, package_connectors:Mini_DIN_6_TE_Connectivity, symbol Connector:Mini-DIN-6
- removed Q1, Q2: NPN, Package_TO_SOT_THT:TO-92_HandSolder, symbol Device:Q_NPN_BCE
- removed R11, R12: 5K, Resistor_THT:R_Axial_DIN0204_L3.6mm_D1.6mm_P5.08mm_Horizontal, symbol Device:R
- removed U12: 74HC245, Package_DIP:DIP-20_W7.62mm_Socket, symbol 74xx:74HC245
- removed U9: 74LS04, Package_DIP:DIP-14_W7.62mm_Socket, symbol 74xx:74LS04
- added J4: 8 Bit Output, Connector_PinHeader_2.54mm:PinHeader_2x07_P2.54mm_Vertical, symbol Connector_Generic:Conn_02x07_Odd_Even
- added J6: FT_232 B, Connector_PinHeader_2.54mm:PinHeader_1x06_P2.54mm_Vertical, symbol Connector_Generic:Conn_01x06
- added J7: Enable Lines, Connector_PinHeader_2.54mm:PinHeader_1x08_P2.54mm_Vertical, symbol Connector_Generic:Conn_01x08
- added JP7: 7Seg Enable, Connector_PinHeader_2.54mm:PinHeader_1x02_P2.54mm_Vertical, symbol Jumper:Jumper_2_Open
- added R16, R17, R18, R19, R20, R21: 330, Resistor_THT:R_Axial_DIN0207_L6.3mm_D2.5mm_P10.16mm_Horizontal, symbol Device:R
- added R22: 1k, Resistor_THT:R_Axial_DIN0207_L6.3mm_D2.5mm_P10.16mm_Horizontal, symbol Device:R
- added R23, R24, R25: 2K, Resistor_THT:R_Axial_DIN0207_L6.3mm_D2.5mm_P10.16mm_Horizontal, symbol Device:R
- added unit 4 of U1
- added U13: 74LS573, Package_DIP:DIP-20_W7.62mm_Socket, symbol 74xx:74LS573
- added unit 5 of U5
- added U9: 74LS32, Package_DIP:DIP-14_W7.62mm_Socket, symbol 74xx:74LS32
- C10, C8, C9: renamed from C?; footprint (none) -> Capacitor_THT:C_Disc_D4.3mm_W1.9mm_P5.00mm
- C7: footprint Capacitor_THT:C_Disc_D3.0mm_W2.0mm_P2.50mm -> Capacitor_THT:C_Disc_D4.3mm_W1.9mm_P5.00mm
- J1: value FT_232 -> FT_232 A
- J1_5VtoSerial1: value Conn_01x02 -> 5V Serial
- J3: value 8 Bit Port -> 8 Bit Input; symbol Connector_Generic:Conn_02x07_Top_Bottom -> Connector_Generic:Conn_02x07_Odd_Even
- R1, R10, R2, R3, R5, R6, R7, R8, R9: footprint Resistor_THT:R_Axial_DIN0204_L3.6mm_D1.6mm_P5.08mm_Horizontal -> Resistor_THT:R_Axial_DIN0207_L6.3mm_D2.5mm_P10.16mm_Horizontal
- R11, R12: renamed from R?; footprint (none) -> Resistor_THT:R_Axial_DIN0207_L6.3mm_D2.5mm_P10.16mm_Horizontal
- R13, R14: value 5K -> 330; footprint Resistor_THT:R_Axial_DIN0204_L3.6mm_D1.6mm_P5.08mm_Horizontal -> Resistor_THT:R_Axial_DIN0207_L6.3mm_D2.5mm_P10.16mm_Horizontal
- R15: footprint (none) -> Resistor_THT:R_Axial_DIN0207_L6.3mm_D2.5mm_P10.16mm_Horizontal
- R4: value 220 -> 1k; footprint Resistor_THT:R_Axial_DIN0204_L3.6mm_D1.6mm_P5.08mm_Horizontal -> Resistor_THT:R_Axial_DIN0207_L6.3mm_D2.5mm_P10.16mm_Horizontal
- SW1: renamed from SW?; footprint (none) -> Button_Switch_THT:Push_E-Switch_KS01Q01
- U1: footprint Package_DIP:DIP-14_W7.62mm -> Package_DIP:DIP-14_W7.62mm_Socket
- U2: footprint Package_DIP:DIP-40_W15.24mm -> Package_DIP:DIP-40_W15.24mm_Socket
- gave numbers to parts that had none: 1
Connections:
- net labels added: AO0, AO1, AO2, AO3, DI0, DI1, DI2, DI3, DI4, DI5, DI6, DI7, DO0, DO1, DO2, DO3, DO4, DO5, DO6, DO7, Y0_WR, ~Y5~, ~Y6~, ~Y7~
- net labels removed: IO0, IO1, IO2, IO3, IO4, IO5, IO6, IO7, KEY_CLK, KEY_DATA, RD, TODO_INVERT_RESET, Y1, ~IOREQ~
- wire segments 419 -> 432
Other:
- note added: "IEI for graphics chip?"
- note added: "Y0 = 7Seg, 8 Bit In/Out\nY1 = Unused\nY2 = Serial\nY3 = CTC\nY4 = PS/2"
- note added: "for output too"
- note removed: "Y0 = 7Seg\nY1 = 8 Bit In/Out\nY2 = Serial\nY3 = CTC\nY4 = PS/2"
- moved on the sheet: C1, C10, C2, C8, C9, J1, J1_5VtoSerial1, J3, JP1, JP2, JP3, JP4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

Commit message: Schema
Parts:
- removed C7: 100nF, Capacitor_THT:C_Disc_D4.3mm_W1.9mm_P5.00mm, symbol Device:C
- removed J3: 8 Bit Input, Connector_PinHeader_2.54mm:PinHeader_2x07_P2.54mm_Vertical, symbol Connector_Generic:Conn_02x07_Odd_Even
- removed U10: 5161AS, 7seg:7SegmentLED_LTS6760_LTS6780, symbol 7seg:5161AS
- added C11, C12, C15, C16, C17: 100n, Capacitor_THT:C_Disc_D4.3mm_W1.9mm_P5.00mm, symbol Device:C
- added C13, C14: 4.7u, Capacitor_THT:C_Radial_D6.3mm_H5.0mm_P2.50mm, symbol Device:C
- added D1: POWER, LED_THT:LED_D3.0mm, symbol Device:LED
- added J10: JACK_TRS, dtz80:Tayda_3.5mm_stereo_TRS_jack_A-853, symbol dtZ80:JACK_TRS
- added J11: YM Parallel IO, Connector_PinHeader_2.54mm:PinHeader_2x09_P2.54mm_Vertical, symbol Connector_Generic:Conn_02x09_Odd_Even
- added J12: Micro USB, Connector_PinHeader_2.54mm:PinHeader_1x05_P2.54mm_Vertical, symbol Connector_Generic:Conn_01x05
- added J13, J14, J15, J16, J17, J18, J19, J20, J21, J22: Conn_01x01, MountingHole:MountingHole_3.2mm_M3_DIN965_Pad, symbol Connector_Generic:Conn_01x01
- added J3: LCD Display, Connector_PinHeader_2.54mm:PinHeader_1x16_P2.54mm_Vertical, symbol Connector_Generic:Conn_01x16
- added J8: External Clock, Connector_PinHeader_2.54mm:PinHeader_1x03_P2.54mm_Vertical, symbol Connector_Generic:Conn_01x03
- added J9: System Bus, Connector_PinHeader_2.54mm:PinHeader_2x20_P2.54mm_Vertical, symbol Connector_Generic:Conn_02x20_Odd_Even
- added JP8: Auto Reset, Connector_PinHeader_2.54mm:PinHeader_1x02_P2.54mm_Vertical, symbol Jumper:Jumper_2_Open
- added JP9: IEI External, Connector_PinHeader_2.54mm:PinHeader_1x02_P2.54mm_Vertical, symbol Jumper:Jumper_2_Open
- added R26, R27, R28: 3k, Resistor_THT:R_Axial_DIN0207_L6.3mm_D2.5mm_P10.16mm_Horizontal, symbol Device:R
- added R29, R30, R31, R32: 1k, Resistor_THT:R_Axial_DIN0207_L6.3mm_D2.5mm_P10.16mm_Horizontal, symbol Device:R
- added R33: 330, Resistor_THT:R_Axial_DIN0207_L6.3mm_D2.5mm_P10.16mm_Horizontal, symbol Device:R
- added RV1: R_POT, Potentiometer_THT:Potentiometer_ACP_CA9-V10_Vertical, symbol Device:R_POT
- added U10: 5161AS, dtz80:7SegmentLED_LTS6760_LTS6780, symbol dtZ80:5161AS
- added U14: YM2149, Package_DIP:DIP-40_W15.24mm_Socket, symbol Audio:YM2149
- added U15: 74HCT138, Package_DIP:DIP-16_W7.62mm_Socket, symbol 74xx:74LS138
- added U16: 74HC00, Package_DIP:DIP-14_W7.62mm_Socket, symbol 74xx:74HC00
- added unit 6 of U5
- added unit 5 of U9
- J2: symbol Connector:Conn_01x05_Male -> Connector_Generic:Conn_01x05
- JP5: value X1 -> X1 Clock
- JP6: value Y1 -> Y1 Clock
- R1, R10: value 1k -> 10k
- SW1: footprint Button_Switch_THT:Push_E-Switch_KS01Q01 -> Button_Switch_THT:SW_TH_Tactile_Omron_B3F-10xx
- U3: footprint dtZ80-main:DIP-28_W15.24mm_Socket_Large_Holes -> dtz80:DIP-28_W15.24mm_Socket_Large_Holes
Connections:
- net labels added: BC1, BDIR, DIO0, DIO1, DIO2, DIO3, DIO4, DIO5, DIO6, DIO7, IEI, IOA0, IOA1, IOA2, IOA3, IOA4, IOA5, IOA6, IOA7, IOB0, IOB1, IOB2, IOB3, IOB4, IOB5, IOB6, IOB7, RXA, TXA, V0
- net labels removed: DI0, DI1, DI2, DI3, DI4, DI5, DI6, DI7, DO0, DO1, DO2, DO3, DO4, DO5, DO6, DO7, RX, TX
- wire segments 432 -> 593
- no-connect marks 30 -> 41
Other:
- note added: "A0 does not conflict with Y0?"
- note added: "Y0 = 7Seg, 8 Bit In/Out\nY1 = Unused\nY2 = Serial\nY3 = CTC\nY4 = Sound Base address\n"
- note added: "disable if u8 enabled?"
- note removed: "TODO:\nWR in 138?"
- note removed: "Y0 = 7Seg, 8 Bit In/Out\nY1 = Unused\nY2 = Serial\nY3 = CTC\nY4 = PS/2"
- moved on the sheet: R10, U1E, U4C, U5G

Commit message: Schema completet
Parts:
- added JP10: ROM On, Connector_PinHeader_2.54mm:PinHeader_1x02_P2.54mm_Vertical, symbol Jumper:Jumper_2_Open
- added JP11: ROM Off, Connector_PinHeader_2.54mm:PinHeader_1x02_P2.54mm_Vertical, symbol Jumper:Jumper_2_Open
- added R34: 10k, Resistor_THT:R_Axial_DIN0207_L6.3mm_D2.5mm_P10.16mm_Horizontal, symbol Device:R
Connections:
- wire segments 593 -> 598
- no-connect marks 41 -> 44
Changed lines of the file:
@@
 Text Label 3750 8000 0    50   ~ 0
 A15
-Text Label 2500 5000 0    50   ~ 0
+Text Label 1950 5400 0    50   ~ 0
 A15
 Wire Wire Line
@@
 	2750 4500 2500 4500
 Wire Wire Line
-	2500 5000 2750 5000
+	1950 5400 2200 5400
 Wire Wire Line
 	3050 9200 3050 9350
@@
 Text Label 11200 10300 3    50   ~ 0
 TXA
-Text Label 12150 900  1    50   ~ 0
-RXA
-Text Label 12150 1550 1    50   ~ 0
-TXA
 Text Label 11500 10300 3    50   ~ 0
 ~Y7~
@@
 	1    0    0    -1
 $EndComp
+NoConn ~ 12150 700
+NoConn ~ 12150 1600
+$Comp
+L Jumper:Jumper_2_Open JP10
+U 1 1 609A9B49
+P 2400 5400
+F 0 "JP10" H 2400 5635 50  0000 C CNN
+F 1 "ROM On" H 2400 5544 50  0000 C CNN
+F 2 "Connector_PinHeader_2.54mm:PinHeader_1x02_P2.54mm_Vertical" H 2400 5400 50  0001 C CNN
+F 3 "~" H 2400 5400 50  0001 C CNN
+	1    2400 5400
+	1    0    0    -1
+$EndComp
+$Comp
+L Jumper:Jumper_2_Open JP11
+U 1 1 60AC66EE
+P 2400 5600
+F 0 "JP11" H 2400 5835 50  0000 C CNN
+F 1 "ROM Off" H 2400 5450 50  0000 C CNN
+F 2 "Connector_PinHeader_2.54mm:PinHeader_1x02_P2.54mm_Vertical" H 2400 5600 50  0001 C CNN
+F 3 "~" H 2400 5600 50  0001 C CNN
+	1    2400 5600
+	1    0    0    -1
+$EndComp
+Connection ~ 2600 5400
+Wire Wire Line
+	2600 5400 2600 5600
+Wire Wire Line
+	2200 5600 1950 5600
+$Comp
+L Device:R R34
+U 1 1 60C6BA80
+P 1800 5600
+F 0 "R34" H 1870 5646 50  0000 L CNN
+F 1 "10k" H 1870 5555 50  0000 L CNN
+F 2 "Resistor_THT:R_Axial_DIN0207_L6.3mm_D2.5mm_P10.16mm_Horizontal" V 1730 5600 50  0001 C CNN
+F 3 "~" H 1800 5600 50  0001 C CNN
+	1    1800 5600
+	0    1    1    0
+$EndComp
+Wire Wire Line
+	1650 5600 1450 5600
+$Comp
+L power:+5V #PWR0114
+U 1 1 60C6CEB9
+P 1450 5600
+F 0 "#PWR0114" H 1450 5450 50  0001 C CNN
+F 1 "+5V" H 1465 5773 50  0000 C CNN
+F 2 "" H 1450 5600 50  0001 C CNN
+F 3 "" H 1450 5600 50  0001 C CNN
+	1    1450 5600
+	1    0    0    -1
+$EndComp
+Wire Wire Line
+	2750 5000 2600 5000
+Wire Wire Line
+	2600 5000 2600 5400
+NoConn ~ 15350 13950
 $EndSCHEMATC

Commit message: gerber files
Other:
- note removed: "A0 does not conflict with Y0?"
Changed lines of the file:
@@
 	0    1    1    0
 $EndComp
-Text Notes 8350 8350 0    50   ~ 0
-A0 does not conflict with Y0?
 Wire Wire Line
 	5450 6950 5450 7150
